File: blubaru/_saved_control.sch (KiCad schematic (older format))
At the start: 1 part, among them J4 ProMicro

Commit message: Create footprints for breakout boards
Parts:
- J4: footprint (none) -> blubaru:ProMicro
Changed lines of the file:
@@
 F 0 "J4" H 5550 3300 60  0000 C CNN
 F 1 "ProMicro" H 5550 4600 60  0000 C CNN
-F 2 "" H 5550 4600 60  0001 C CNN
+F 2 "blubaru:ProMicro" H 5550 4600 60  0001 C CNN
 F 3 "" H 5550 4600 60  0001 C CNN
 	1    5550 4600
