File: blubaru/control.sch (KiCad schematic (older format))
At the start: 1 part, among them J4 ProMicro

Commit message: Put parts in the audio switch page.
Changed lines of the file:
@@
 $EndComp
 $Comp
-L GND #PWR07
+L GND #PWR010
 U 1 1 589BF3A5
 P 6400 4200
-F 0 "#PWR07" H 6400 3950 50  0001 C CNN
+F 0 "#PWR010" H 6400 3950 50  0001 C CNN
 F 1 "GND" H 6400 4050 50  0000 C CNN
 F 2 "" H 6400 4200 50  0000 C CNN
@@
 $EndComp
 $Comp
-L GND #PWR08
+L GND #PWR011
 U 1 1 589BF4DD
 P 4750 4400
-F 0 "#PWR08" H 4750 4150 50  0001 C CNN
+F 0 "#PWR011" H 4750 4150 50  0001 C CNN
 F 1 "GND" H 4750 4250 50  0000 C CNN
 F 2 "" H 4750 4400 50  0000 C CNN
@@
 $EndComp
 $Comp
-L VCC #PWR09
+L VCC #PWR012
 U 1 1 589BF5FE
-P 4500 4200
-F 0 "#PWR09" H 4500 4050 50  0001 C CNN
-F 1 "VCC" H 4500 4350 50  0000 C CNN
-F 2 "" H 4500 4200 50  0000 C CNN
-F 3 "" H 4500 4200 50  0000 C CNN
-	1    4500 4200
+P 4750 4200
+F 0 "#PWR012" H 4750 4050 50  0001 C CNN
+F 1 "VCC" H 4750 4350 50  0000 C CNN
+F 2 "" H 4750 4200 50  0000 C CNN
+F 3 "" H 4750 4200 50  0000 C CNN
+	1    4750 4200
 	1    0    0    -1
 $EndComp
@@
 	4750 4400 5050 4400
 Wire Wire Line
-	4500 4200 5050 4200
+	4750 4200 5050 4200
 Wire Wire Line
 	5050 4750 5050 4500
@@
 	6050 4400 6550 4400
 $Comp
-L +12V #PWR010
+L +12V #PWR013
 U 1 1 58B175C7
 P 5050 4750
-F 0 "#PWR010" H 5050 4600 50  0001 C CNN
+F 0 "#PWR013" H 5050 4600 50  0001 C CNN
 F 1 "+12V" H 5050 4890 50  0000 C CNN
 F 2 "" H 5050 4750 50  0000 C CNN
