File: blubaru/bt.sch (KiCad schematic (older format))
At the start: 3 parts, among them J2 RN52_BREAKOUT, P1 CONN_01X06

Commit message: Put parts in the audio switch page.
Parts:
- renumbered C12 to C1, J2 to J5
Changed lines of the file:
@@
 $EndDescr
 $Comp
-L RN52_BREAKOUT J2
+L RN52_BREAKOUT J5
 U 1 1 589AA2F8
 P 5100 2950
-F 0 "J2" H 5100 850 60  0000 C CNN
+F 0 "J5" H 5100 850 60  0000 C CNN
 F 1 "RN52_BREAKOUT" H 5100 2950 60  0000 C CNN
 F 2 "" H 5100 2950 60  0001 C CNN
@@
 $EndComp
 $Comp
-L GND #PWR011
+L GND #PWR014
 U 1 1 589AA392
 P 5800 5250
-F 0 "#PWR011" H 5800 5000 50  0001 C CNN
+F 0 "#PWR014" H 5800 5000 50  0001 C CNN
 F 1 "GND" H 5800 5100 50  0000 C CNN
 F 2 "" H 5800 5250 50  0000 C CNN
@@
 $EndComp
 $Comp
-L VCC #PWR012
+L VCC #PWR015
 U 1 1 589AA3E5
 P 4400 5250
-F 0 "#PWR012" H 4400 5100 50  0001 C CNN
+F 0 "#PWR015" H 4400 5100 50  0001 C CNN
 F 1 "VCC" H 4400 5400 50  0000 C CNN
 F 2 "" H 4400 5250 50  0000 C CNN
@@
 NoConn ~ 5800 3950
 $Comp
-L C C12
+L C C1
 U 1 1 589BA198
 P 5100 5250
-F 0 "C12" H 5125 5350 50  0000 L CNN
+F 0 "C1" H 5125 5350 50  0000 L CNN
 F 1 "0.1uF" H 5125 5150 50  0000 L CNN
 F 2 "" H 5138 5100 50  0000 C CNN
@@
 $EndComp
 $Comp
-L GND #PWR013
+L GND #PWR016
 U 1 1 589E813D
 P 3950 3350
-F 0 "#PWR013" H 3950 3100 50  0001 C CNN
+F 0 "#PWR016" H 3950 3100 50  0001 C CNN
 F 1 "GND" H 3950 3200 50  0000 C CNN
 F 2 "" H 3950 3350 50  0000 C CNN
@@
 	3850 3350 3950 3350
 Wire Wire Line
-	5800 3050 6800 2900
-Wire Wire Line
-	5800 3150 6800 3000
-Wire Wire Line
-	5800 3250 6800 3100
-Wire Wire Line
-	5800 3350 6800 3200
+	5800 3050 6700 3050
+Wire Wire Line
+	5800 3150 6700 3150
+Wire Wire Line
+	5800 3250 6700 3250
+Wire Wire Line
+	5800 3350 6700 3350
 $Sheet
-S 6800 3550 750  600
+S 7000 3900 750  600
 U 58AE7D2D
 F0 "Microphone" 60
 F1 "mic.sch" 60
-F2 "MIC_R-" O L 6800 3650 60
-F3 "MIC_L-" O L 6800 3750 60
-F4 "MIC_R+" O L 6800 3850 60
-F5 "MIC_L+" O L 6800 3950 60
-F6 "MIC_BIAS" O L 6800 4050 60
+F2 "MIC_R-" O L 7000 4000 60
+F3 "MIC_L-" O L 7000 4100 60
+F4 "MIC_R+" O L 7000 4200 60
+F5 "MIC_L+" O L 7000 4300 60
+F6 "MIC_BIAS" O L 7000 4400 60
 $EndSheet
-Wire Wire Line
-	5800 3450 6800 3650
-Wire Wire Line
-	5800 3550 6800 3750
-Wire Wire Line
-	5800 3650 6800 3850
-Wire Wire Line
-	5800 3750 6800 3950
-Wire Wire Line
-	5800 3850 6800 4050
 $Sheet
-S 6800 2800 1100 500
+S 6700 2950 1100 500
 U 58AE00D8
 F0 "Amp" 60
 F1 "amp.sch" 60
-F2 "LineOutL" O R 7900 2900 60
-F3 "LineOutR" O R 7900 3000 60
-F4 "L+" I L 6800 2900 60
-F5 "R+" I L 6800 3000 60
-F6 "L-" I L 6800 3100 60
-F7 "R-" I L 6800 3200 60
+F2 "LineOutL" O R 7800 3050 60
+F3 "LineOutR" O R 7800 3150 60
+F4 "L+" I L 6700 3050 60
+F5 "R+" I L 6700 3150 60
+F6 "L-" I L 6700 3250 60
+F7 "R-" I L 6700 3350 60
 $EndSheet
-Text HLabel 8250 2900 2    60   Output ~ 0
+Text HLabel 8150 3050 2    60   Output ~ 0
 LineOutL
-Text HLabel 8250 3000 2    60   Output ~ 0
+Text HLabel 8150 3150 2    60   Output ~ 0
 LineOutR
 Wire Wire Line
-	7900 2900 8250 2900
-Wire Wire Line
-	7900 3000 8250 3000
+	7800 3050 8150 3050
+Wire Wire Line
+	7800 3150 8150 3150
 Text HLabel 4000 4450 0    60   Output ~ 0
 UART_TX
@@
 Wire Wire Line
 	4100 3950 4400 3950
+Wire Wire Line
+	5800 3450 6550 3450
+Wire Wire Line
+	5800 3550 6450 3550
+Wire Wire Line
+	5800 3650 6350 3650
+Wire Wire Line
+	5800 3750 6250 3750
+Wire Wire Line
+	5800 3850 6150 3850
+Wire Wire Line
+	6550 3450 6550 4000
+Wire Wire Line
+	6550 4000 7000 4000
+Wire Wire Line
+	6450 3550 6450 4100
+Wire Wire Line
+	6450 4100 7000 4100
+Wire Wire Line
+	6350 3650 6350 4200
+Wire Wire Line
+	6350 4200 7000 4200
+Wire Wire Line
+	6250 3750 6250 4300
+Wire Wire Line
+	6250 4300 7000 4300
+Wire Wire Line
+	6150 3850 6150 4400
+Wire Wire Line
+	6150 4400 7000 4400
 $EndSCHEMATC

Commit message: Create footprints for breakout boards
Parts:
- C1: footprint (none) -> Capacitors_THT:C_Disc_D5.0mm_W2.5mm_P2.50mm
- P1: footprint (none) -> Pin_Headers:Pin_Header_Straight_1x06_Pitch2.54mm
Changed lines of the file:
@@
 encoding utf-8
 Sheet 6 8
-Title ""
-Date ""
+Title "Blubaru"
+Date "2017-02-28"
 Rev ""
 Comp ""
@@
 $EndComp
 $Comp
-L GND #PWR014
+L GND #PWR017
 U 1 1 589AA392
 P 5800 5250
-F 0 "#PWR014" H 5800 5000 50  0001 C CNN
+F 0 "#PWR017" H 5800 5000 50  0001 C CNN
 F 1 "GND" H 5800 5100 50  0000 C CNN
 F 2 "" H 5800 5250 50  0000 C CNN
@@
 $EndComp
 $Comp
-L VCC #PWR015
+L VCC #PWR018
 U 1 1 589AA3E5
 P 4400 5250
-F 0 "#PWR015" H 4400 5100 50  0001 C CNN
+F 0 "#PWR018" H 4400 5100 50  0001 C CNN
 F 1 "VCC" H 4400 5400 50  0000 C CNN
 F 2 "" H 4400 5250 50  0000 C CNN
@@
 F 0 "C1" H 5125 5350 50  0000 L CNN
 F 1 "0.1uF" H 5125 5150 50  0000 L CNN
-F 2 "" H 5138 5100 50  0000 C CNN
+F 2 "Capacitors_THT:C_Disc_D5.0mm_W2.5mm_P2.50mm" H 5138 5100 50  0001 C CNN
 F 3 "" H 5100 5250 50  0000 C CNN
 	1    5100 5250
@@
 F 0 "P1" H 3650 3950 50  0000 C CNN
 F 1 "CONN_01X06" V 3750 3600 50  0000 C CNN
-F 2 "" H 3650 3600 50  0000 C CNN
+F 2 "Pin_Headers:Pin_Header_Straight_1x06_Pitch2.54mm" H 3650 3600 50  0001 C CNN
 F 3 "" H 3650 3600 50  0000 C CNN
 	1    3650 3600
@@
 $EndComp
 $Comp
-L GND #PWR016
+L GND #PWR019
 U 1 1 589E813D
 P 3950 3350
-F 0 "#PWR016" H 3950 3100 50  0001 C CNN
+F 0 "#PWR019" H 3950 3100 50  0001 C CNN
 F 1 "GND" H 3950 3200 50  0000 C CNN
 F 2 "" H 3950 3350 50  0000 C CNN

Commit message: Actually save the schematics that I had open.
Parts:
- J5: footprint (none) -> blubaru:RN52_Breakout
Changed lines of the file:
@@
 F 0 "J5" H 5100 850 60  0000 C CNN
 F 1 "RN52_BREAKOUT" H 5100 2950 60  0000 C CNN
-F 2 "" H 5100 2950 60  0001 C CNN
+F 2 "blubaru:RN52_Breakout" H 5100 2950 60  0001 C CNN
 F 3 "" H 5100 2950 60  0001 C CNN
 	1    5100 2950
