File: blubaru/blubaru.kicad_pcb (KiCad board)
At the start: 2 copper layers, 97.8 x 94.6 mm, 38 parts, among them J1 DB15, J2 DB15, J3 FSA2269, J4 ProMicro, J5 RN52_BREAKOUT, J6 JACK_TRS_6PINS, J7 TPA6112, P1 CONN_01X06, U1 DG419

Commit message: Added footprint for audio jack.
Connections:
- J1 pad 15: (no net) -> Net-(J1-Pad15)
- J2 pad 15: (no net) -> Net-(J2-Pad15)
- J4 pad 10: (no net) -> Net-(J4-Pad10)
- J4 pad 11: (no net) -> Net-(J4-Pad11)
- J4 pad 13: (no net) -> Net-(J4-Pad13)
- J4 pad 14: (no net) -> Net-(J4-Pad14)
- J4 pad 15: (no net) -> Net-(J4-Pad15)
- J4 pad 16: (no net) -> Net-(J4-Pad16)
- J4 pad 17: (no net) -> Net-(J4-Pad17)
- J4 pad 18: (no net) -> Net-(J4-Pad18)
- J4 pad 19: (no net) -> Net-(J4-Pad19)
- J4 pad 20: (no net) -> Net-(J4-Pad20)
- J4 pad 22: (no net) -> Net-(J4-Pad22)
- J4 pad 7: (no net) -> Net-(J4-Pad7)
- J4 pad 8: (no net) -> Net-(J4-Pad8)
- J4 pad 9: (no net) -> Net-(J4-Pad9)
- J5 pad 1: (no net) -> Net-(J5-Pad1)
- J5 pad 11: (no net) -> Net-(J5-Pad11)
- J5 pad 12: (no net) -> Net-(J5-Pad12)
- J5 pad 13: (no net) -> Net-(J5-Pad13)
- J5 pad 14: (no net) -> Net-(J5-Pad14)
- J5 pad 17: (no net) -> Net-(J5-Pad17)
- J5 pad 18: (no net) -> Net-(J5-Pad18)
- J5 pad 22: (no net) -> Net-(J5-Pad22)
- J5 pad 23: (no net) -> Net-(J5-Pad23)
- J5 pad 24: (no net) -> Net-(J5-Pad24)
- J5 pad 25: (no net) -> Net-(J5-Pad25)
- J5 pad 26: (no net) -> Net-(J5-Pad26)
- J5 pad 27: (no net) -> Net-(J5-Pad27)
- J5 pad 28: (no net) -> Net-(J5-Pad28)
- J5 pad 29: (no net) -> Net-(J5-Pad29)
- J5 pad 3: (no net) -> Net-(J5-Pad3)
- J5 pad 30: (no net) -> Net-(J5-Pad30)
- J5 pad 31: (no net) -> Net-(J5-Pad31)
- J5 pad 4: (no net) -> Net-(J5-Pad4)
- J6 pad 4: (no net) -> Net-(J6-Pad4)
- J6 pad 5: (no net) -> Net-(J6-Pad5)
- J6 pad 6: (no net) -> Net-(J6-Pad6)
