File: modules.sch (KiCad schematic (older format))
At the start: 2 parts

Commit message: Add LEDs to MCU and polarized caps on line driver.
Parts:
- removed D1: LED, symbol LED
- removed R1: R, Resistors_THT:R_Axial_DIN0204_L3.6mm_D1.6mm_P1.90mm_Vertical, symbol R
Changed lines of the file:
@@
 Wire Wire Line
 	4650 4900 5500 4900
-$Comp
-L R R1
-U 1 1 58D327F2
-P 5300 3850
-F 0 "R1" V 5380 3850 50  0000 C CNN
-F 1 "R" V 5300 3850 50  0000 C CNN
-F 2 "Resistors_THT:R_Axial_DIN0204_L3.6mm_D1.6mm_P1.90mm_Vertical" V 5230 3850 50  0001 C CNN
-F 3 "" H 5300 3850 50  0001 C CNN
-	1    5300 3850
-	1    0    0    -1
-$EndComp
-$Comp
-L LED D1
-U 1 1 58D32887
-P 5300 4200
-F 0 "D1" H 5300 4300 50  0000 C CNN
-F 1 "LED" H 5300 4100 50  0000 C CNN
-F 2 "" H 5300 4200 50  0001 C CNN
-F 3 "" H 5300 4200 50  0001 C CNN
-	1    5300 4200
-	0    -1   -1   0
-$EndComp
-$Comp
-L GND #PWR07
-U 1 1 58D32928
-P 5300 4400
-F 0 "#PWR07" H 5300 4150 50  0001 C CNN
-F 1 "GND" H 5300 4250 50  0000 C CNN
-F 2 "" H 5300 4400 50  0001 C CNN
-F 3 "" H 5300 4400 50  0001 C CNN
-	1    5300 4400
-	1    0    0    -1
-$EndComp
-Wire Wire Line
-	5300 3650 5300 3700
-Connection ~ 5300 3650
-Wire Wire Line
-	5300 4000 5300 4050
-Wire Wire Line
-	5300 4350 5300 4400
 $EndSCHEMATC

Commit message: Add an LED indicator to the trigger
Parts:
- added D?: LED, symbol LED
- added R?: R, symbol R
Connections:
- net Audio switch/BT_TRG: now also R?.1
- new net: D?.2 (A), R?.2
- new net GND: D?.1 (K)
Changed lines of the file:
@@
 Wire Wire Line
 	4650 4900 5500 4900
+$Comp
+L R R?
+U 1 1 58D327F2
+P 5300 3850
+F 0 "R?" V 5380 3850 50  0000 C CNN
+F 1 "R" V 5300 3850 50  0000 C CNN
+F 2 "" V 5230 3850 50  0001 C CNN
+F 3 "" H 5300 3850 50  0001 C CNN
+	1    5300 3850
+	1    0    0    -1
+$EndComp
+$Comp
+L LED D?
+U 1 1 58D32887
+P 5300 4200
+F 0 "D?" H 5300 4300 50  0000 C CNN
+F 1 "LED" H 5300 4100 50  0000 C CNN
+F 2 "" H 5300 4200 50  0001 C CNN
+F 3 "" H 5300 4200 50  0001 C CNN
+	1    5300 4200
+	0    -1   -1   0
+$EndComp
+$Comp
+L GND #PWR?
+U 1 1 58D32928
+P 5300 4400
+F 0 "#PWR?" H 5300 4150 50  0001 C CNN
+F 1 "GND" H 5300 4250 50  0000 C CNN
+F 2 "" H 5300 4400 50  0001 C CNN
+F 3 "" H 5300 4400 50  0001 C CNN
+	1    5300 4400
+	1    0    0    -1
+$EndComp
+Wire Wire Line
+	5300 3650 5300 3700
+Connection ~ 5300 3650
+Wire Wire Line
+	5300 4000 5300 4050
+Wire Wire Line
+	5300 4350 5300 4400
 $EndSCHEMATC

Commit message: Add a line_driver schematic
This branch contains the full line driver with 2nd order filter, which
provides a low-pass filter on the input.
Parts:
- gave numbers to parts that had none: 2
Changed lines of the file:
@@
 	4650 4900 5500 4900
 $Comp
-L R R?
+L R R1
 U 1 1 58D327F2
 P 5300 3850
-F 0 "R?" V 5380 3850 50  0000 C CNN
+F 0 "R1" V 5380 3850 50  0000 C CNN
 F 1 "R" V 5300 3850 50  0000 C CNN
 F 2 "" V 5230 3850 50  0001 C CNN
@@
 $EndComp
 $Comp
-L LED D?
+L LED D1
 U 1 1 58D32887
 P 5300 4200
-F 0 "D?" H 5300 4300 50  0000 C CNN
+F 0 "D1" H 5300 4300 50  0000 C CNN
 F 1 "LED" H 5300 4100 50  0000 C CNN
 F 2 "" H 5300 4200 50  0001 C CNN
@@
 $EndComp
 $Comp
-L GND #PWR?
+L GND #PWR07
 U 1 1 58D32928
 P 5300 4400
-F 0 "#PWR?" H 5300 4150 50  0001 C CNN
+F 0 "#PWR07" H 5300 4150 50  0001 C CNN
 F 1 "GND" H 5300 4250 50  0000 C CNN
 F 2 "" H 5300 4400 50  0001 C CNN

Commit message: add component values and footprints.
Parts:
- R1: footprint (none) -> Resistors_THT:R_Axial_DIN0204_L3.6mm_D1.6mm_P1.90mm_Vertical
Changed lines of the file:
@@
 F 0 "R1" V 5380 3850 50  0000 C CNN
 F 1 "R" V 5300 3850 50  0000 C CNN
-F 2 "" V 5230 3850 50  0001 C CNN
+F 2 "Resistors_THT:R_Axial_DIN0204_L3.6mm_D1.6mm_P1.90mm_Vertical" V 5230 3850 50  0001 C CNN
 F 3 "" H 5300 3850 50  0001 C CNN
 	1    5300 3850
