File: line_in.sch (KiCad schematic (older format))
At the start: 4 parts, among them J9 JACK_TRS_5PINS

Commit message: Reduce the line driver back to simple
After determining the gain needed to be 0.735 (which is out of spec for
the amp), I was unsure what to do with the 2nd order filter on the amp.
It wasn't even present on the headphone amp from before, and I suspect
the head unit in the car does some filtering of its own. To simplify
things, I removed the second order filter and went back to a simple line
driver. I also set the values of the gain setting resistors to 8.2 and
11, which gets as close as I can to 0.735 gain using single E24
resistors.
Parts:
- renumbered R19 to R13, R20 to R14, R21 to R15
Changed lines of the file:
@@
 $EndComp
 $Comp
-L GND #PWR037
+L GND #PWR035
 U 1 1 595D4619
 P 6150 3700
-F 0 "#PWR037" H 6150 3450 50  0001 C CNN
+F 0 "#PWR035" H 6150 3450 50  0001 C CNN
 F 1 "GND" H 6150 3550 50  0000 C CNN
 F 2 "" H 6150 3700 50  0001 C CNN
@@
 	4400 3350 6300 3350
 $Comp
-L R R19
+L R R13
 U 1 1 595F0365
 P 5200 2950
-F 0 "R19" V 5280 2950 50  0000 C CNN
+F 0 "R13" V 5280 2950 50  0000 C CNN
 F 1 "100k" V 5200 2950 50  0000 C CNN
 F 2 "Resistors_THT:R_Axial_DIN0204_L3.6mm_D1.6mm_P5.08mm_Horizontal" V 5130 2950 50  0001 C CNN
@@
 $EndComp
 $Comp
-L GND #PWR038
+L GND #PWR036
 U 1 1 595F03CA
 P 5200 2750
-F 0 "#PWR038" H 5200 2500 50  0001 C CNN
+F 0 "#PWR036" H 5200 2500 50  0001 C CNN
 F 1 "GND" H 5200 2600 50  0000 C CNN
 F 2 "" H 5200 2750 50  0001 C CNN
@@
 Connection ~ 5850 3600
 $Comp
-L GND #PWR039
+L GND #PWR037
 U 1 1 595F0532
 P 5200 3750
-F 0 "#PWR039" H 5200 3500 50  0001 C CNN
+F 0 "#PWR037" H 5200 3500 50  0001 C CNN
 F 1 "GND" H 5200 3600 50  0000 C CNN
 F 2 "" H 5200 3750 50  0001 C CNN
@@
 $EndComp
 $Comp
-L R R20
+L R R14
 U 1 1 595F054E
 P 5200 3550
-F 0 "R20" V 5280 3550 50  0000 C CNN
+F 0 "R14" V 5280 3550 50  0000 C CNN
 F 1 "100k" V 5200 3550 50  0000 C CNN
 F 2 "Resistors_THT:R_Axial_DIN0204_L3.6mm_D1.6mm_P5.08mm_Horizontal" V 5130 3550 50  0001 C CNN
@@
 	5850 3450 5850 4050
 $Comp
-L R R21
+L R R15
 U 1 1 595F0435
 P 5650 3600
-F 0 "R21" V 5730 3600 50  0000 C CNN
+F 0 "R15" V 5730 3600 50  0000 C CNN
 F 1 "1M" V 5650 3600 50  0000 C CNN
 F 2 "Resistors_THT:R_Axial_DIN0204_L3.6mm_D1.6mm_P5.08mm_Horizontal" V 5580 3600 50  0001 C CNN
@@
 	5450 3600 5500 3600
 $Comp
-L VCC #PWR040
+L VCC #PWR038
 U 1 1 5971D586
 P 5450 3550
-F 0 "#PWR040" H 5450 3400 50  0001 C CNN
+F 0 "#PWR038" H 5450 3400 50  0001 C CNN
 F 1 "VCC" H 5450 3700 50  0000 C CNN
 F 2 "" H 5450 3550 50  0001 C CNN

Commit message: Separate audio ground from power ground
The connection between the CD player and stereo has a separate line for
audio ground and the chassis ground. I didn't previously understand why
this was necessary, so I tied them together. They were tied together in
the stereo anyway. The reason is that when using power, there must be
current returning on the ground line, and since that ground line is not
free of resistance, that causes a slight voltage change. That voltage
difference causes a disagreement in what ground is, and at audio levels,
that makes a significant difference. By isolating the audio ground to a
separate wire that doesn't carry current, we keep the ground potential
the same between the devices, and the audio comes out much cleaner.

On the main connector, I've kept the chassis ground as the power ground,
and only connected the audio ground to the mid-rail on the line driver,
and the line-in ground, as those are the places where audio ground
potential will matter.

As I now understand the grounding situation better, I'm removing the
ground jumper pads.

I will also consider removing the voltage regulator if I can get enough
power out of the regulator on board with the MCU.
Connections:
- net GND: no longer J9.1 (S)
- new net GNDA: J9.1 (S)
Changed lines of the file:
@@
 	-1   0    0    1
-$EndComp
-$Comp
-L GND #PWR035
-U 1 1 595D4619
-P 6150 3700
-F 0 "#PWR035" H 6150 3450 50  0001 C CNN
-F 1 "GND" H 6150 3550 50  0000 C CNN
-F 2 "" H 6150 3700 50  0001 C CNN
-F 3 "" H 6150 3700 50  0001 C CNN
-	1    6150 3700
-	1    0    0    -1
 $EndComp
 Wire Wire Line
@@
 $EndComp
 $Comp
-L GND #PWR036
+L GND #PWR035
 U 1 1 595F03CA
 P 5200 2750
-F 0 "#PWR036" H 5200 2500 50  0001 C CNN
+F 0 "#PWR035" H 5200 2500 50  0001 C CNN
 F 1 "GND" H 5200 2600 50  0000 C CNN
 F 2 "" H 5200 2750 50  0001 C CNN
@@
 Connection ~ 5850 3600
 $Comp
-L GND #PWR037
+L GND #PWR036
 U 1 1 595F0532
 P 5200 3750
-F 0 "#PWR037" H 5200 3500 50  0001 C CNN
+F 0 "#PWR036" H 5200 3500 50  0001 C CNN
 F 1 "GND" H 5200 3600 50  0000 C CNN
 F 2 "" H 5200 3750 50  0001 C CNN
@@
 	5450 3600 5500 3600
 $Comp
-L VCC #PWR038
+L VCC #PWR037
 U 1 1 5971D586
 P 5450 3550
-F 0 "#PWR038" H 5450 3400 50  0001 C CNN
+F 0 "#PWR037" H 5450 3400 50  0001 C CNN
 F 1 "VCC" H 5450 3700 50  0000 C CNN
 F 2 "" H 5450 3550 50  0001 C CNN
@@
 	1    0    0    -1
 $EndComp
+$Comp
+L GNDA #PWR038
+U 1 1 59C09A2F
+P 6150 3700
+F 0 "#PWR038" H 6150 3450 50  0001 C CNN
+F 1 "GNDA" H 6150 3550 50  0000 C CNN
+F 2 "" H 6150 3700 50  0000 C CNN
+F 3 "" H 6150 3700 50  0000 C CNN
+	1    6150 3700
+	1    0    0    -1
+$EndComp
