File: control.sch (KiCad schematic (older format))
At the start: 17 parts, among them IC1 ATTINY4313-P, P2 CONN_02X03, SW1 SW_Push, Y1 11.0592MHz

Commit message: First full layout
I renumbered pins on the MCU so that the layout was cleaner, hence the
regenerated net file.

This passes all the design rules and nothing is unconnected. I managed
to get the ground pour connected without having to pour between pins,
but it seems even better connected if I do, and it is within the design
rules, so it seems safe.
Changed lines of the file:
@@
 Text HLabel 6800 4900 2    60   Output ~ 0
 UART_RX
-Text HLabel 6800 3900 2    60   Output ~ 0
+Text HLabel 6800 5200 2    60   Output ~ 0
 CMD
-Text HLabel 6800 5000 2    60   Input ~ 0
+Text HLabel 6800 5100 2    60   Input ~ 0
 EVENT
-Text HLabel 6800 5200 2    60   Output ~ 0
+Text HLabel 6800 4000 2    60   Output ~ 0
 BT_TRG
 $Comp
@@
 	0    1    1    0
 $EndComp
-Text HLabel 6800 5300 2    60   Output ~ 0
+Text HLabel 6800 4100 2    60   Output ~ 0
 LINE_TRG
 Wire Wire Line
 	6300 4200 6800 4200
-Text HLabel 6800 5100 2    60   Input ~ 0
+Text HLabel 6800 3900 2    60   Input ~ 0
 JACK_SENSE
 Wire Wire Line
@@
 Wire Wire Line
 	8800 4700 8800 4750
+Text HLabel 6800 5000 2    60   Output ~ 0
+BT_RESET
+Wire Wire Line
+	6300 3900 6800 3900
 Text HLabel 6800 5400 2    60   Output ~ 0
-BT_RESET
-Wire Wire Line
-	6300 3900 6800 3900
-Text HLabel 6800 4100 2    60   Output ~ 0
 PWR_EN
 Wire Wire Line
@@
 Wire Wire Line
 	6300 4100 6800 4100
-Text HLabel 6800 4000 2    60   Output ~ 0
+Text HLabel 6800 5300 2    60   Output ~ 0
 9600
 Wire Wire Line
@@
 Wire Wire Line
 	6300 5400 6800 5400
+Text Label 6600 4300 2    60   ~ 0
+LED1
 Text Label 6600 4200 2    60   ~ 0
-LED1
-Text Label 6600 4300 2    60   ~ 0
 LED2
-Text Label 6650 5200 2    60   ~ 0
+Text Label 6650 4000 2    60   ~ 0
 BT_TRG
-Text Label 6700 5300 2    60   ~ 0
+Text Label 6700 4100 2    60   ~ 0
 LINE_TRG
 Wire Wire Line
