File: blubaru.kicad_pcb (KiCad board)
At the start: 2 copper layers, 80 x 79.5 mm, 68 parts, among them IC1 ATTINY4313-P, J1 DB15, J2 DB15, J3 TS5A22364-Q1, J4 TS5A22364-Q1, J5 RN52_BREAKOUT, J6 JACK_TRS_5PINS, J7 DRV632, J8 JACK_TRS_5PINS, P1 CONN_01X06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

Commit message: Add some logos to the back.
Parts:
- added REF**: KiCAD Logo, Symbols:Symbol_KiCAD-Logo_CopperAndSilkScreenTop, B.Cu at (152.9, 106.7)
- added REF***: OSHW-Logo_11.4x12mm_SilkScreen, Symbols:OSHW-Logo_11.4x12mm_SilkScreen, B.Cu at (185.2, 111.8)
- added REF***: ESD-Logo_6.6x6mm_SilkScreen, Symbols:ESD-Logo_6.6x6mm_SilkScreen, B.Cu at (123.3, 112.6)
- added REF***: WEEE-Logo_4.2x6mm_SilkScreen, Symbols:WEEE-Logo_4.2x6mm_SilkScreen, B.Cu at (186.7, 133.3)
Other:
- board text added: "CD"
- board text added: "Stereo"
